File: EAGLE/ha-pc-switch/ha-pc-switch-revA.brd (EAGLE design)
At the start: 88.9 x 43.2 mm, 85 parts, among them J4 QWIIC_RIGHT_ANGLE, Q1 NPN, Q2 NPN, Q3 NPN, Q4 NPN, U1 STM8S001J3, U2 ILD213T, U3 ILD213T, U5 ILD213T, U6 ILD213T, U7 REG1117-3.3

Commit message: _
Parts:
- removed D3, D4: (no value), adafruit:SOD-523
- added R33: 0R, rcl:R0603
Connections:
- removed net N$10: D4.A, J3.1
- new net VXX: J3.1, R33.2, U1.4
- net VCC: now also R33.1; no longer D3.A
- net V_ISOL: no longer D3.K, D4.K, U1.4
Changed lines of the file:
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@@
 <drawing>
 <settings>
-<setting alwaysvectorfont="yes"/>
+<setting alwaysvectorfont="no"/>
 <setting verticaltext="up"/>
 </settings>
-<grid distance="50" unitdist="mil" unit="mil" style="lines" multiple="1" display="yes" altdistance="5" altunitdist="mil" altunit="mil"/>
+<grid distance="1" unitdist="mm" unit="mm" style="dots" multiple="1" display="yes" altdistance="0.1" altunitdist="mm" altunit="mm"/>
 <layers>
 <layer number="1" name="Top" color="4" fill="1" visible="yes" active="yes"/>
@@
 <attribute name="VALUE" x="184.46" y="32.6792" size="1.27" layer="27"/>
 </element>
-<element name="D3" library="adafruit" library_urn="urn:adsk.eagle:library:420" package="SOD-523" package3d_urn="urn:adsk.eagle:package:6240751/1" value="" x="178" y="41" smashed="yes">
-<attribute name="NAME" x="179.016" y="42.016" size="0.4064" layer="25"/>
-<attribute name="VALUE" x="179.016" y="39.476" size="0.4064" layer="27"/>
-</element>
-<element name="D4" library="adafruit" library_urn="urn:adsk.eagle:library:420" package="SOD-523" package3d_urn="urn:adsk.eagle:package:6240751/1" value="" x="178" y="37" smashed="yes">
-<attribute name="NAME" x="179.016" y="38.016" size="0.4064" layer="25"/>
-<attribute name="VALUE" x="179.016" y="35.476" size="0.4064" layer="27"/>
-</element>
 <element name="D1" library="adafruit" library_urn="urn:adsk.eagle:library:420" package="SOD-523" package3d_urn="urn:adsk.eagle:package:6240751/1" value="" x="178" y="33" smashed="yes">
 <attribute name="NAME" x="179.016" y="34.016" size="0.4064" layer="25"/>
@@
 <attribute name="PROD_ID" value="Combine 8288+8399" x="110" y="49" size="1.778" layer="27" display="off"/>
 <attribute name="VALUE" x="115.334" y="50.524" size="0.6096" layer="27" font="vector" ratio="20"/>
+</element>
+<element name="R33" library="rcl" library_urn="urn:adsk.eagle:library:334" package="R0603" package3d_urn="urn:adsk.eagle:package:23555/3" value="0R" x="2" y="-3" smashed="yes">
+<attribute name="NAME" x="1.365" y="-2.365" size="1.27" layer="25"/>
+<attribute name="POPULARITY" value="70" x="2" y="-3" size="1.778" layer="27" display="off"/>
+<attribute name="SPICEPREFIX" value="R" x="2" y="-3" size="1.778" layer="27" display="off"/>
+<attribute name="VALUE" x="1.365" y="-4.905" size="1.27" layer="27"/>
 </element>
 </elements>
@@
 <contactref element="R27" pad="2"/>
 <contactref element="R28" pad="2"/>
-<contactref element="D3" pad="A"/>
 <contactref element="ESP-12F" pad="VCC"/>
 <contactref element="C6" pad="1"/>
@@
 <contactref element="R20" pad="2"/>
 <contactref element="R24" pad="2"/>
+<contactref element="R33" pad="1"/>
 <wire x1="189.311" y1="30.901" x2="195.5" y2="34" width="0" layer="19" extent="1-1"/>
 <wire x1="187" y1="30.901" x2="189.311" y2="30.901" width="0" layer="19" extent="1-1"/>
 <wire x1="187" y1="37.099" x2="187" y2="30.901" width="0" layer="19" extent="1-1"/>
-<wire x1="178" y1="40.2" x2="187" y2="37.099" width="0" layer="19" extent="1-1"/>
-<wire x1="171.85" y1="42" x2="178" y2="40.2" width="0" layer="19" extent="1-1"/>
-<wire x1="171.85" y1="32" x2="171.85" y2="42" width="0" layer="19" extent="1-1"/>
-<wire x1="171.85" y1="27" x2="171.85" y2="32" width="0" layer="19" extent="1-1"/>
-<wire x1="171.85" y1="22" x2="171.85" y2="27" width="0" layer="19" extent="1-1"/>
-<wire x1="178.15" y1="24" x2="171.85" y2="22" width="0" layer="19" extent="1-1"/>
+<wire x1="178.15" y1="24" x2="187" y2="30.901" width="0" layer="19" extent="1-1"/>
 <wire x1="178.15" y1="19" x2="178.15" y2="24" width="0" layer="19" extent="1-1"/>
 <wire x1="178.15" y1="14" x2="178.15" y2="19" width="0" layer="19" extent="1-1"/>
 <wire x1="178.15" y1="9" x2="178.15" y2="14" width="0" layer="19" extent="1-1"/>
+<wire x1="171.85" y1="22" x2="178.15" y2="24" width="0" layer="19" extent="1-1"/>
+<wire x1="171.85" y1="27" x2="171.85" y2="22" width="0" layer="19" extent="1-1"/>
+<wire x1="171.85" y1="32" x2="171.85" y2="27" width="0" layer="19" extent="1-1"/>
+<wire x1="171.85" y1="42" x2="171.85" y2="32" width="0" layer="19" extent="1-1"/>
 <wire x1="157.26" y1="37.09" x2="171.85" y2="42" width="0" layer="19" extent="1-1"/>
 <wire x1="136.94" y1="37.09" x2="157.26" y2="37.09" width="0" layer="19" extent="1-1"/>
@@
 <wire x1="27.55" y1="17.8" x2="31.756" y2="36.83" width="0" layer="19" extent="1-1"/>
 <wire x1="31.756" y1="13.97" x2="27.55" y2="17.8" width="0" layer="19" extent="1-1"/>
+<wire x1="1.15" y1="-3" x2="27.55" y2="17.8" width="0" layer="19" extent="1-1"/>
 </signal>
 <signal name="T_PWR_SWT">
@@
 <wire x1="24.136" y1="13.97" x2="23.55" y2="17.8" width="0" layer="19" extent="1-1"/>
 </signal>
-<signal name="N$10">
-<contactref element="J3" pad="1"/>
-<contactref element="D4" pad="A"/>
-<wire x1="178" y1="36.2" x2="135" y2="13" width="0" layer="19" extent="1-1"/>
-</signal>
 <signal name="V_ISOL">
-<contactref element="U1" pad="4"/>
 <contactref element="C2" pad="1"/>
-<contactref element="D3" pad="K"/>
-<contactref element="D4" pad="K"/>
-<wire x1="122.44" y1="19.31" x2="145.996" y2="5.975" width="0" layer="19" extent="1-1"/>
-<wire x1="178" y1="41.8" x2="122.44" y2="19.31" width="0" layer="19" extent="1-1"/>
-<wire x1="178" y1="37.8" x2="178" y2="41.8" width="0" layer="19" extent="1-1"/>
 </signal>
 <signal name="SWIM">
@@
 <wire x1="170.15" y1="7" x2="16.516" y2="36.83" width="0" layer="19" extent="1-1"/>
 </signal>
+<signal name="VXX">
+<contactref element="J3" pad="1"/>
+<contactref element="U1" pad="4"/>
+<contactref element="R33" pad="2"/>
+<wire x1="135" y1="13" x2="145.996" y2="5.975" width="0" layer="19" extent="1-1"/>
+<wire x1="2.85" y1="-3" x2="135" y2="13" width="0" layer="19" extent="1-1"/>
+</signal>
 </signals>

Commit message: _
Parts:
- removed J1, J_HDD_LED_3, J_PC_ON_1, J_PC_ON_3, J_PWR_LED_1, J_PWR_LED_2, UNDEF_1, UNDEF_2: (no value), SparkFun-Connectors:1X02_NO_SILK
- removed J2: (no value), SparkFun-Connectors:SCREWTERMINAL-3.5MM-5
- removed J4: QWIIC_RIGHT_ANGLE, ts_custom_nick_nacks:JST04_1MM_RA
- removed J_PC_ON_2, J_PWR_LED2: (no value), SparkFun-Connectors:1X02_LONGPADS
- removed LOGO2: OSHW-LOGOM, random_logos:OSHW-LOGO-M
- removed S1: (no value), ts_custom_nick_nacks:SKRKAEE020
- removed U$6: TECSMITH-LOGOLONG, random_logos:TECSMITH-NAME
- removed U6: ILD213T, SparkFun:SO08-2
- added J_HDD_LED_2, J_MSG_LED_1, J_MSG_LED_2, J_NC_1, J_NC_2, J_PWR_1, J_PWR_2, RST: (no value), SparkFun-Connectors:1X02_NO_SILK
- added J_MSG_LED_3, J_PWR_3: (no value), SparkFun-Connectors:1X02_LONGPADS
- added J_OPT: (no value), SparkFun-Connectors:SCREWTERMINAL-3.5MM-5
- added J_QWIIC: QWIIC_RIGHT_ANGLE, ts_custom_nick_nacks:JST04_1MM_RA
- added S_RST: (no value), ts_custom_nick_nacks:SKRKAEE020
- added TP1, TP2, TP3, TP4, TP5, TP6, TP7, TP8: TEST-POINT3X5, SparkFun-Connectors:PAD.03X.05
- added U$5: MOUNTINGHOLE3.0THIN, ts_custom_nick_nacks:MOUNTINGHOLE_3.0_PLATEDTHIN
- added U4: TLP3123, __untitled:SOP4_TOS
- C1: value 470nF -> 100nF
- C2: value 100nF -> 470nF
- C3, C4: value 100nF -> 330uF
- C7, C9: value 330uF -> 100nF
- J_RESET_2: device SparkFun-Connectors:1X02_LONGPADS -> SparkFun-Connectors:1X02_NO_SILK
- J_RESET_3: device SparkFun-Connectors:1X02_NO_SILK -> SparkFun-Connectors:1X02_LONGPADS
- R13, R15: value 10 -> 220R
- R14, R16: value 220R -> 10R
- R2: value 10K -> 220R
- R22: value 10K -> 0R
- R23: value 0R -> 10K
- R25: value 330R -> 0R
- R26: value 10K -> 330R
- R30: value 330R -> 10K
- R33: value 0R -> 330R
- R4: value 220R -> 10K
- U5: value ILD213T -> TLP3123; device SparkFun:SO08-2 -> __untitled:SOP4_TOS
- moved R33 169.1 mm to (171.0, 2.00)
- moved U$9 102.7 mm to (9.40, 4.82)
- moved J_RESET_2 81.9 mm to (73.7, 34.3), turned to 90 degrees
- moved U$12 80.8 mm to (86.0, 4.83)
- moved U$11 80.1 mm to (91.9, 4.84)
- moved C4 69.1 mm to (179.0, 9.00)
- moved C7 67.4 mm to (112.0, 25.7)
- moved J_PSU_2 66.5 mm to (66.2, 41.3), turned to 180 degrees
- moved J_RESET_1 66.0 mm to (83.8, 34.3), turned to 90 degrees
- moved C3 60.6 mm to (179.0, 14.0)
- moved C6 59.4 mm to (119.6, 25.7)
- moved J_PSU_1 54.1 mm to (64.8, 44.5), turned to 180 degrees
- moved J_RESET_3 49.6 mm to (94.0, 35.6), turned to 270 degrees
- moved R4 34.7 mm to (125.9, 37.1)
- moved J_HDD_LED_1 33.2 mm to (83.8, 41.9), turned to 270 degrees
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- renumbered J3 to STM8_SWIM
Connections:
- removed net V_ISOL: C2.1
- new net VDD: C4.1, C8.1, C9.1, D1-MINI.3V3, ESP-12F.VCC, ESP-PROG_2X3.2, J_OPT.3, J_QWIIC.2, R10.2, R11.2, R12.2, R20.2, R21.2, R22.1, R27.2, R28.2, R29.2, R3.2, R4.2, R5.2, R6.2, R9.2, TP2.1, U7.2, U7.T
- net !X_PWR_LONG: now also R33.1, TP8.1; no longer R32.1
- net !X_PWR_SHRT: now also R25.2, R28.1, TP4.1; no longer R23.2, R27.1
- net !X_RST_SHRT: now also TP5.1
- net 5VIN: now also R2.1; no longer R4.1
- net D1_SCL: now also J_OPT.5, J_QWIIC.4; no longer J2.5, J4.4
- net D2_SDA: now also J_OPT.4, J_QWIIC.3; no longer J2.4, J4.3
- net ESP_EN: now also R27.1; no longer R26.1
- net ESP_IO0: now also R29.1, R33.2; no longer R28.1, R32.2
- net GND: now also C3.2, C4.2, J_OPT.2, J_QWIIC.1, R23.1, R24.1, R30.1, RST.2, S_RST.2, TP3.1, U4.2; no longer C6.2, C7.2, J1.2, J2.2, J4.1, R21.1, R22.1, R29.1, S1.2, U5.4, U6.2, U6.4
- net HDD_LED+: now also J_HDD_LED_2.1; no longer J_HDD_LED_3.1
- net HDD_LED-: now also J_HDD_LED_2.2; no longer J_HDD_LED_3.2
- net N$14: now also R26.2; no longer R25.2
- net N$15: now also R32.2; no longer R31.2
- net N$16: now also R31.2; no longer R30.2
- net N$2: now also R2.2; no longer R4.2
- net N$24: now also C2.1; no longer C1.1
- net N$3: now also J_NC_1.1, J_NC_2.1; no longer UNDEF_1.1, UNDEF_2.1
- net N$4: now also J_NC_1.2, J_NC_2.2; no longer UNDEF_1.2, UNDEF_2.2
- net N$5: now also R15.2; no longer R14.2, U5.3
- net N$7: now also C6.1, R14.1; no longer C3.1, R13.1
- net N$8: now also C7.1, R16.1; no longer C4.1, R15.1
- net N$9: now also R13.2, U4.1; no longer R16.2, U6.1, U6.3
- net OUT1N: now also R3.1; no longer R2.1
- net OUT1N1: now also Q3.1; no longer Q4.1
- net OUT2N: now also R4.1; no longer R5.1
- net OUT2N1: now also Q4.1; no longer Q3.1
- net PC_ON+: now also J_PWR_1.1, J_PWR_2.1, J_PWR_3.1, R14.2, U4.4; no longer J_PC_ON_1.1, J_PC_ON_2.1, J_PC_ON_3.1, R13.2, U5.5, U5.8
- net PC_ON-: now also C6.2, J_PWR_1.2, J_PWR_2.2, J_PWR_3.2, U4.3; no longer C3.2, J_PC_ON_1.2, J_PC_ON_2.2, J_PC_ON_3.2, U5.6, U5.7
- net PWR_LED+: now also J_MSG_LED_1.1, J_MSG_LED_2.1, J_MSG_LED_3.1; no longer J_PWR_LED2.2, J_PWR_LED_1.1, J_PWR_LED_2.2
- net PWR_LED-: now also J_MSG_LED_1.2, J_MSG_LED_2.2, J_MSG_LED_3.2; no longer J_PWR_LED2.1, J_PWR_LED_1.2, J_PWR_LED_2.1
- net RESET+: now also R16.2, U5.4; no longer R15.2, U6.5, U6.8
- net RESET-: now also C7.2, U5.3; no longer C4.2, U6.6, U6.7
- net RST: now also R21.1, R26.1, RST.1, S_RST.1; no longer J1.1, R24.1, R25.1, S1.1
- net RX: now also R32.1; no longer R31.1
- net SWIM: now also R25.1; no longer R23.1
- net S_5VIN: now also R5.1; no longer R6.1
- net S_HDD_LED: now also Q4.3; no longer Q3.3
- net S_PWR_LED: now also Q3.3; no longer Q4.3
- net S_PWR_OK: now also R30.2, R6.1; no longer R29.2, R3.1
- net TX: now also R31.1; no longer R30.1
- net T_PWR_SWT: now also R13.1, R23.2, TP6.1; no longer R14.1, R21.2
- net T_RST_SWT: now also R15.1, R24.2, TP7.1; no longer R16.1, R22.2
- net VCC: now also C3.1, J_OPT.1, TP1.1; no longer C6.1, C7.1, C8.1, C9.1, D1-MINI.3V3, ESP-12F.VCC, ESP-PROG_2X3.2, J2.1, J2.3, J4.2, R10.2, R11.2, R12.2, R2.2, R20.2, R24.2, R26.2, R27.2, R28.2, R3.2, R33.1, R5.2, R6.2, R9.2, U7.2, U7.T
- net VXX: now also C1.1, R22.2; no longer R33.2
Other:
- board size 88.9 x 43.2 mm -> 88.9 x 44.4 mm
- board text added: "CHANGE GRID TO 50mil W/ 5mil STEPS"

Commit message: _
Parts:
- removed STM8_SWIM: (no value), SparkFun-Connectors:MOLEX-1X4
- removed TP4, TP5, TP6, TP7, TP8: TEST-POINT3X5, SparkFun-Connectors:PAD.03X.05
- added C10, C11: 12pF, rcl:C0603
- added D3, D4: GREEN, SparkFun-LED:LED-0603
- added J1: 1X04_SMD_STRAIGHT_COMBO, SparkFun-Connectors:1X04_SMD_VERTICAL_COMBO
- added R34: 1K, rcl:R0603
- added TP10, TP11, TP12, TP14, TP15, TP16, TP9: TEST-POINT3X5, SparkFun-Connectors:PAD.03X.05
- added U$15, U$16: FIDUCIAL, adafruit:FIDUCIAL_1MM
- added U$20: ARGB, __temp_to_delete:ARGB
- added U$21: 74AHCT1G125GW, ts_keyboards:SC-88A__TSSOP5__SOT353-1
- added U$22: JUMPER-1X3-CLOSED-2, ts_jumpers:SOLDERJUMPER_CLOSEDWIRE-3-2
- added U$4: NUCLEO_HEADER, stm32c0:NUCLEO
- added Y1: 32.768kHz, SparkFun-Clocks:CRYSTAL-SMD-3.2X1.5MM
- C1: device rcl:C0805 -> rcl:C0603
- C2: value 470nF -> 4.7uF; device rcl:C0805 -> rcl:C0603
- R21: value 10K -> 220R
- R22: value 0R -> 470R
- R25: value 0R -> 1K
- U1: value STM8S001J3 -> STM32C011FTSSOP20_STM-M; device __untitled:SOIC-8 -> stm32c0:TSSOP20-M
- moved R21 182.9 mm to (2.00, -28.0)
- moved R23 167.1 mm to (2.00, -38.0)
- moved R25 166.3 mm to (2.00, -54.0)
- moved R24 165.0 mm to (2.00, -43.0)
- moved R22 140.7 mm to (2.00, -23.0)
- moved U1 70.4 mm to (173.0, 74.0)
- moved C1 59.8 mm to (162.0, 65.0)
- moved C2 51.9 mm to (162.0, 60.0)
Connections:
- removed net D1_SCL: D1-MINI.D1, ESP-12F.GPIO5, J_OPT.5, J_QWIIC.4
- removed net D2_SDA: D1-MINI.D2, ESP-12F.GPIO4, J_OPT.4, J_QWIIC.3
- removed net N$24: C2.1, U1.3
- removed net RX: D1-MINI.RX, ESP-PROG_2X3.5, R32.1
- removed net SWIM: R25.1, STM8_SWIM.2
- removed net VXX: C1.1, R22.2, STM8_SWIM.1, U1.4
- new net A0: D1-MINI.A0, ESP-12F.ADC0, TP12.1
- new net CTS2: U1.16
- new net D1/SCL: D1-MINI.D1, ESP-12F.GPIO5, J_OPT.5, J_QWIIC.4, R23.1, U1.20
- new net D2/SDA: D1-MINI.D2, ESP-12F.GPIO4, J_OPT.4, J_QWIIC.3, R24.1, U1.1
- new net IO10: ESP-12F.GPIO10, TP15.1
- new net IO11: ESP-12F.CS0, TP14.1
- new net IO16: ESP-12F.GPIO16
- new net IO6: ESP-12F.SCLK, TP11.1
- new net IO7: ESP-12F.MISO, TP10.1
- new net IO8: ESP-12F.MOSI, TP9.1
- new net IO9: ESP-12F.GPIO9, TP16.1
- new net N$10: C10.1, U1.2, Y1.P$2
- new net N$11: C11.1, U1.3, Y1.P$1
- new net N$12: R21.2, U$21.2
- new net N$17: R22.1, U$21.4
- new net N$18: R22.2, U$20.D
- new net N$19: D3.A, R25.1
- new net N$20: R23.2, U$22.2
- new net N$21: R24.2, U$22.1
- new net N$25: D4.A, R34.1
- new net RESET: U$4.6, U1.6
- new net RTS2: U1.17
- new net RX/RGB: D1-MINI.RX, ESP-PROG_2X3.5, R21.1, R32.1, U1.15
- new net RX2: U1.8
- new net SWCLK: J1.2, U$4.4, U1.19
- new net SWDIO: J1.3, U$4.2, U1.18
- new net TX2: U1.7
- new net WAKE: U1.11
- net !X_PWR_LONG: now also U1.12; no longer TP8.1, U1.1
- net !X_PWR_SHRT: now also U1.13; no longer R25.2, TP4.1, U1.8
- net !X_RST_SHRT: now also U1.14; no longer TP5.1, U1.7
- net GND: now also C10.2, C11.2, D3.C, D4.C, J1.1, U$20.G, U$21.1, U$21.3, U$4.1, U1.5; no longer R23.1, R24.1, STM8_SWIM.3, U1.2
- net RST: no longer R21.1, STM8_SWIM.4
- net T_PWR_SWT: now also R25.2, U1.10; no longer R23.2, TP6.1, U1.6
- net T_RST_SWT: now also R34.2, U1.9; no longer R24.2, TP7.1, U1.5
- net VCC: now also C1.1, C2.1, J1.4, U$20.V, U$21.6, U$22.3, U$4.3, U1.4
- net VDD: no longer R21.2, R22.1
