File: EAGLE/ha-pc-switch/ha-pc-switch-revB.brd (EAGLE design)
At the start: 70 x 68 mm, 66 parts, among them Y1 32.768kHz

Commit message: _
Parts:
- added TP10, TP6, TP7, TP8, TP9: TPTP16SQ, testpad:TP16SQ
- moved U$16 2.54 mm to (2.54, 58.4)
Connections:
- net T_PWR_SWT: now also TP9.TP
- net T_RST_SWT: now also TP10.TP
- net X_PWR_LONG: now also TP8.TP
- net X_PWR_SHRT: now also TP7.TP
- net X_RST_SHRT: now also TP6.TP
Routing:
- net T_RST_SWT: track 45.6 -> 53.8 mm
- net T_PWR_SWT: track 55.4 -> 62.3 mm
- net X_PWR_LONG: track 42.1 -> 47.6 mm, vias 4 -> 5
- net X_PWR_SHRT: track 39.8 -> 44.9 mm, vias 2 -> 3
- net X_RST_SHRT: track 43.8 -> 47.6 mm, vias 2 -> 3
- net VCC_1: track 165.9 -> 163.7 mm
Other:
- board text added: ">PL"
- board text added: ">PS"
- board text added: ">RS"
- board text added: "Pull-ups"
- board text added: "Pwr>"
- board text added: "Rst>"
