File: EAGLE/ha-pc-switch/ha-pc-switch-revB.sch (EAGLE design)
At the start: 109 parts, among them Q1 NPN, Q2 NPN, Q3 NPN, Q4 NPN, Y1 32.768kHz

Commit message: Rev B
Parts:
- removed ARGB, SCL, SDA: JUMPER-1X3-CLOSED, ts_jumpers:JUMPER-1X3-CLOSED
- removed D1, D2: (no value), adafruit:DIODESOD-523
- removed D1-MINI: LOLIN-D1-MINI-PRO, ts_dev_boards:LOLIN-D1-MINI-PRO
- removed ESP-12F: (no value), ts_dev_boards:ESPRESSIF-ESP-12F&ESMD
- removed J_ARGB: ARGB, __temp_to_delete:ARGB
- removed J_DBG2: NUCLEO_HEADER, stm32c0:NUCLEO_HEADER
- removed J_I2C: (no value), SparkFun-Connectors:CONN_05SCREW
- removed J_MSG_LED_3, J_PWR_3, J_RESET_3: (no value), SparkFun-Connectors:CONN_02PTH3
- removed J_NC_1, J_NC_2, RST: (no value), SparkFun-Connectors:CONN_021X02_NO_SILK
- removed J_PRG1: (no value), SparkFun-Connectors:CONN_03X2FEMALE_SMD
- removed J_PSU_1: (no value), SparkFun-Connectors:CONN_04LONGPADS
- removed J_PSU_2: (no value), SparkFun-Connectors:CONN_04SCREW
- removed J_RGB_5V: JUMPER-1X3-CLOSEDPINS, ts_jumpers:JUMPER-1X3-CLOSEDPINS
- removed LSHFT: 74AHCT1G125GW, ts_keyboards:74AHCT1G125GW
- removed OC_LED, OC_PWR: ILD213T, SparkFun:OPTOISOLATOR-2SOIC8
- removed Q1, Q2, Q3, Q4: NPN, SparkFun:TRANSISTOR_NPNSOT23-3
- removed R19, R20, R27, R28, R29, R30, R9: 10K, rcl:R-EU_R0603
- removed R22: 470R, rcl:R-EU_R0603
- removed R25, R34: 1K, rcl:R-EU_R0603
- removed R26, R31, R32, R33: 330R, rcl:R-EU_R0603
- removed S_RST: (no value), ts_custom_nick_nacks:MOMENTARY-SWITCH-SPST-1
- removed TP1, TP10, TP11, TP12, TP14, TP15, TP16, TP2, TP3, TP4, TP9: TEST-POINT3X5, SparkFun-Connectors:TEST-POINT3X5
- removed U$12, U$5: MOUNTINGHOLE3.0THIN, ts_custom_nick_nacks:MOUNTINGHOLE3.0THIN
- removed VREG: REG1117-3.3, ts_custom_nick_nacks:REG1117-3.3
- added ESP-12: (no value), ts_dev_boards:ESPRESSIF-ESP-12F&ESMD
- added J_BOOT1, J_BOOT2, J_CI_1, J_CI_2, J_RST1, J_RST2: (no value), SparkFun-Connectors:CONN_021X02_NO_SILK
- added J_PRG_1: (no value), SparkFun-Connectors:CONN_03X2NO_SILK
- added LED3, LED4: GREEN, SparkFun-LED:LED-GREEN0603
- added LOGO2: QWIIC_LOGO_4MM, SparkFun-Aesthetics:QWIIC_LOGO_4MM
- added S_BOOT: (no value), ts_custom_nick_nacks:MOMENTARY-SWITCH-SPST-1
- added U$2: PCIE-1X, ts-pcie:PCIE-1X
- C10, C11: value 12pF -> 100nF
- C2: value 4.7uF -> 10uF
- C3, C4: value 330uF -> 100nF
- C5: value 100nF -> 4.7uF
- C7: value 100nF -> 12pF
- C8: value 330uF -> 12pF
- J_PRG2: value 1X04_SMD_STRAIGHT_COMBO -> NUCLEO_HEADER; device SparkFun-Connectors:CONN_04SMD_STRAIGHT_COMBO -> stm32c0:NUCLEO_HEADER
- LED1: value GREEN -> AMBER
- LED2: value GREEN -> BLUE
- R1, R2: value 220R -> 10K
- R14, R16: value 10R -> 1K
- R17, R18: value 10K -> 10R
- R3, R4, R5: value 10K -> 470R
- R7, R8: value 220R -> 1K
Connections:
- removed net !X_PWR_LONG: D1-MINI.D3, R33.1, STM32C0.PA5
- removed net !X_PWR_SHRT: D1-MINI.D4, ESP-12F.2, R28.1, STM32C0.PA6
- removed net !X_RST_SHRT: D1-MINI.D6, ESP-12F.12, R20.1, STM32C0.PA7
- removed net 5VIN: J_PSU_1.4, J_PSU_2.4, J_RGB_5V.1, R2.1
- removed net A0: D1-MINI.A0, ESP-12F.ADC, TP12.1
- removed net ARGB: ARGB.2, LSHFT.A_DIN
- removed net IO10: ESP-12F.10, TP15.1
- removed net IO11: ESP-12F.11, TP14.1
- removed net IO16: ESP-12F.16
- removed net IO6: ESP-12F.6, TP11.1
- removed net IO7: ESP-12F.7, TP10.1
- removed net IO8: ESP-12F.8, TP9.1
- removed net IO9: ESP-12F.9, TP16.1
- removed net N$12: J_ARGB.V, J_RGB_5V.2, LSHFT.5_VCC
- removed net N$13: D1.C, OC_LED.A1, R7.2
- removed net N$17: LSHFT.Y_DOUT, R22.1
- removed net N$18: J_ARGB.D, R22.2
- removed net N$3: J_NC_1.1, J_NC_2.1
- removed net N$4: J_NC_1.2, J_NC_2.2
- removed net N$6: D2.C, OC_LED.A2, R8.2
- removed net OUT1N: OC_PWR.CL1, Q1.B, R3.1
- removed net OUT1N1: OC_LED.CL1, Q3.B, R9.1
- removed net OUT2N: OC_PWR.CL2, Q2.B, R4.1
- removed net OUT2N1: OC_LED.CL2, Q4.B, R10.1
- removed net PWR_OK: J_PSU_1.3, J_PSU_2.3, R1.1
- removed net RESET: J_DBG2.NC, STM32C0.PF2-NRST
- removed net RST: C5.1, D1-MINI.RST, R26.1, RST.1, S_RST.1
- removed net SCL1: D1-MINI.D1, ESP-12F.5, SCL.1
- removed net SDA1: D1-MINI.D2, ESP-12F.4, SDA.1
- removed net S_5VIN: D1-MINI.D7, ESP-12F.13, Q2.C, R19.2, R5.1
- removed net S_HDD_LED: D1-MINI.D5, ESP-12F.14, Q4.C, R11.1, R18.2
- removed net S_PWR_LED: D1-MINI.D0, Q3.C, R12.1, R17.2
- removed net S_PWR_OK: D1-MINI.D8, ESP-12F.15, Q1.C, R30.2, R6.1
- removed net VCC: C3.1, D1-MINI.5V, J_I2C.1, J_PSU_1.2, J_PSU_2.2, J_RGB_5V.3, TP1.1, VREG.IN
- removed net VDD: C1.1, C2.1, C4.1, C8.1, C9.1, D1-MINI.3V3, ESP-12F.VCC, I2C.2, J_DBG2.3V3, J_I2C.3, J_PRG1.2, J_PRG2.4, J_QWIIC.2, R10.2, R11.2, R12.2, R20.2, R27.2, R28.2, R29.2, R3.2, R4.2, R5.2, R6.2, R9.2, STM32C0.VDD/VDDA, TP2.1, VREG.OUT
- new net BOOT: C3.1, ESP-12.0, J_BOOT1.1, S_BOOT.1
- new net CI+: J_CI_1.2, J_CI_2.2
- new net CI-: J_CI_1.1, J_CI_2.1
- new net N$23: ESP-12.TX, R4.2
- new net N$24: ESP-12.15, R6.2
- new net RST1: C4.1, ESP-12.RST, J_RST1.1, R1.1
- new net RST2: C9.1, J_PRG2.NC, J_RST2.1, STM32C0.PF2-NRST
- new net VCC_1: C1.1, C2.1, C5.1, C6.1, ESP-12.VCC, I2C.2, J_PRG2.3V3, J_PRG_1.2, J_QWIIC.2, R1.2, R2.1, R8.2, STM32C0.VDD/VDDA, U$2.3V3AUX-B10
- new net VCC_2: R3.1, R7.2, U$2.3V3-A10, U$2.3V3-A9, U$2.3V3-B8
- new net X_PWR_LONG: ESP-12.13, R12.2, STM32C0.PA5
- new net X_PWR_SHRT: ESP-12.12, R11.2, STM32C0.PA6
- new net X_RST_SHRT: ESP-12.14, R10.2, STM32C0.PA7
- net ESP_EN: now also ESP-12.EN, J_PRG_1.1, R2.2; no longer ESP-12F.EN, J_PRG1.1, R27.1
- net ESP_IO0: now also J_PRG_1.6; no longer ESP-12F.0, J_PRG1.6, R29.1, R33.2
- net GND: now also C6.2, C7.2, ESP-12.GND, J_BOOT1.2, J_BOOT2.2, J_PRG2.GND, J_PRG_1.4, J_RST1.2, J_RST2.2, LED3.C, LED4.C, R10.1, R11.1, R12.1, R6.1, S_BOOT.3, U$2.GND-A12, U$2.GND-A15, U$2.GND-A18, U$2.GND-A4, U$2.GND-B13, U$2.GND-B16, U$2.GND-B18, U$2.GND-B4, U$2.GND-B7; no longer C10.2, C11.2, D1-MINI.GND, ESP-12F.GND, J_ARGB.G, J_DBG2.GND, J_I2C.2, J_PRG1.4, J_PRG2.1, J_PSU_1.1, J_PSU_2.1, LED1.C, LED2.C, LSHFT.!OE, LSHFT.3_GND, OC_LED.EM1, OC_LED.EM2, OC_PWR.C1, OC_PWR.C2, OC_PWR.EM1, OC_PWR.EM2, Q1.E, Q2.E, Q3.E, Q4.E, R17.1, R18.1, R19.1, R30.1, RST.2, S_RST.3, TP3.1, VREG.GND
- net HDD_LED+: no longer R8.1
- net HDD_LED-: no longer D2.A, OC_LED.C2
- net N$1: now also ESP-12.16, R3.2; no longer OC_PWR.A1, R1.2
- net N$10: now also C8.1; no longer C10.1
- net N$11: now also C7.1; no longer C11.1
- net N$14: now also LED1.A, R7.1; no longer ESP-12F.RST, R26.2
- net N$15: now also ESP-12.RX, R5.2; no longer ESP-12F.RX, R32.2
- net N$16: now also ESP-12.2, LED1.C, LED2.C; no longer ESP-12F.TX, R31.2
- net N$19: now also LED3.A, R14.1; no longer LED1.A, R25.1
- net N$2: now also LED2.A, R8.1; no longer OC_PWR.A2, R2.2
- net N$25: now also LED4.A, R16.1; no longer LED2.A, R34.1
- net N$7: now also C10.1, R17.1; no longer C6.1, R14.1
- net N$8: now also C11.1, R18.1; no longer C7.1, R16.1
- net PC_ON+: now also R17.2; no longer J_PWR_3.1, R14.2
- net PC_ON-: now also C10.2; no longer C6.2, J_PWR_3.2
- net PWR_LED+: no longer J_MSG_LED_3.1, R7.1
- net PWR_LED-: no longer D1.A, J_MSG_LED_3.2, OC_LED.C1
- net RESET+: now also R18.2; no longer J_RESET_3.1, R16.2
- net RESET-: now also C11.2; no longer C7.2, J_RESET_3.2
- net RX1: now also J_PRG_1.5, R5.1; no longer ARGB.1, D1-MINI.RX, J_PRG1.5, R32.1
- net SCL: now also ESP-12.5; no longer J_I2C.5, SCL.2
- net SCL2: no longer SCL.3
- net SDA: now also ESP-12.4; no longer J_I2C.4, SDA.2
- net SDA2: no longer SDA.3
- net SWCLK: now also J_BOOT2.1, J_PRG2.SWCLK; no longer J_DBG2.SWCLK, J_PRG2.2
- net SWDIO: now also J_PRG2.SWDIO; no longer J_DBG2.SWDIO, J_PRG2.3
- net TX1: now also J_PRG_1.3, R4.1; no longer D1-MINI.TX, J_PRG1.3, R31.1
- net T_PWR_SWT: now also R14.2; no longer R25.2
- net T_RST_SWT: now also R16.2; no longer R34.2
- net WAKE: no longer TP4.1
- net X_SPARE: no longer ARGB.3
Other:
- note added: "Ai-Thinker ESP-12F / *-12S / *-07 / *C2-12 Module"
- note added: "I2C Pull-Ups"
- note added: "Inter-MCU Pull-Downs"
- note added: "Optional IO"
- note added: "PCIe 1x Slot"
- note added: "STM32C011Fx Relay "One-Shot" Delay-OFF Timer"
- note added: "VCC1 = Always On 3.3V (a.k.a. STANDBY) VCC2 = Only On when PC also On"
- note removed: "5V POWER SOURCE"
- note removed: "5V to 3.3V Regulator for ESP-12F configuration"
- note removed: "ARGB Feature"
- note removed: "Ai-Thinker ESP-12F Module (Alternative)"
- note removed: "Common rest button"
- note removed: "DO NOT POPULATE (Only to be used if not using a D1 Mini)"
- note removed: "Input Sensors"
- note removed: "Optional IO / Expansion headers"
- note removed: "Rvrs Prot"
- note removed: "STM32C011Fx Relay "On-Shot" Delay-OFF Timer"
- note removed: "VCC = 5V (supplied by PSU Standby) VDD = 3.3V (supplied by D1-Mini or opt. LM1117)"
- note removed: "WEMOS / LOLIN D1 Mini Module"

Commit message: _
Parts:
- added TP10, TP6, TP7, TP8, TP9: TPTP16SQ, testpad:TPTP16SQ
Connections:
- net T_PWR_SWT: now also TP9.TP
- net T_RST_SWT: now also TP10.TP
- net X_PWR_LONG: now also TP8.TP
- net X_PWR_SHRT: now also TP7.TP
- net X_RST_SHRT: now also TP6.TP
Other:
- moved on the sheet: J_CI_1, J_CI_2, J_HDD_LED_1, J_HDD_LED_2, J_MSG_LED_1, J_MSG_LED_2, J_PWR_1, J_PWR_2, J_RESET_1, J_RESET_2, LED3, LED4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
